File: Sprinkle/AvionicsV0.kicad_pcb (KiCad board)
At the start: 4 copper layers, 63.5 x 99 mm, 144 parts, among them IC1 ESP32-S3-WROOM-1U-N4R2, IC2 USBLC6-2SC6, IC3 NCP1117IST33T3G, J1 Micro_SD_Card, J10 Conn_01x02, J11 Conn_Coaxial, J12 Conn_01x04, J13 Conn_Coaxial, J14 Conn_01x02, J16 Conn_01x04, J17 Conn_01x06, J2 USB_B_Micro, J3 Conn_01x02, J4 Conn_01x02, J5 Conn_01x02, J6 Conn_01x02, J7 Conn_01x02, J8 Conn_01x02, J9 Conn_01x02, M1 TP6841S6-A, Q1 SIR182DP-T1-RE3, Q2 SIR182DP-T1-RE3, Q3 2N7002H, Q4 SIR182DP-T1-RE3, Q5 SIR182DP-T1-RE3, SW1 SW_Push, SW2 SW_Push, U1 MS8607, U2 LPS22HB, U3 ICM-20649, U4 FGPMMOPA6H, U8 RFM98PW, U9 LSM6DS3

Commit message: Add files via upload
Parts:
- removed the G*** at (152.4, 120.4)
- added C17: 0.1uF, Capacitor_SMD:C_0603_1608Metric, B.Cu at (176.7, 112.5)
- added G***: LOGO, Exo_Bronco_Avionics_Footprints:rocket_image, F.Cu at (151.9, 114.3)
- added R8: 10k, Resistor_SMD:R_0603_1608Metric, B.Cu at (170.2, 114.0)
- added TP10: GPS-RX-UART-TP, TestPoint:TestPoint_Keystone_5000-5004_Miniature, F.Cu at (147.3, 89.7)
- added TP13: SPI-MISO, TestPoint:TestPoint_Keystone_5000-5004_Miniature, F.Cu at (144.6, 79.2)
- added TP14: SPI-MOSI, TestPoint:TestPoint_Keystone_5000-5004_Miniature, F.Cu at (143.5, 89.7)
- added TP15: SPI-CLK, TestPoint:TestPoint_Keystone_5000-5004_Miniature, F.Cu at (124.5, 73.7)
- added TP16: Pyro-MFET4-TP, TestPoint:TestPoint_Pad_D1.0mm, F.Cu at (135.9, 117.8)
- added TP17: Pyro-MFET1-TP, TestPoint:TestPoint_Pad_D1.0mm, F.Cu at (137.9, 125.9)
- added TP18: Pyro-MFET2-TP, TestPoint:TestPoint_Pad_D1.0mm, F.Cu at (137.9, 132.8)
- added TP19: Pyro-MFET2-TP, TestPoint:TestPoint_Pad_D1.0mm, F.Cu at (137.9, 139.9)
- added TP2: GND TP, TestPoint:TestPoint_Keystone_5000-5004_Miniature, F.Cu at (160.1, 144.7)
- added TP20: Pyro-HPO-TP, TestPoint:TestPoint_Pad_D1.0mm, F.Cu at (152.4, 144.6)
- added TP21: Cont-A4-TP, TestPoint:TestPoint_Pad_D1.0mm, F.Cu at (140.3, 125.9)
- added TP22: Cont-A3-TP, TestPoint:TestPoint_Pad_D1.0mm, F.Cu at (140.4, 132.8)
- added TP23: Cont-A2-TP, TestPoint:TestPoint_Pad_D1.0mm, F.Cu at (140.4, 139.9)
- added TP24: Cont-A1-TP, TestPoint:TestPoint_Pad_D1.0mm, F.Cu at (135.9, 147.4)
- added TP3: 3V3 TP, TestPoint:TestPoint_Pad_D1.5mm, F.Cu at (141.5, 120.5)
- added TP4: 5V TP, TestPoint:TestPoint_Pad_D1.5mm, F.Cu at (144.3, 120.5)
- added TP5: Vbus TP, TestPoint:TestPoint_Pad_D1.5mm, F.Cu at (165.4, 121.1)
- added TP6: RG5 TP, TestPoint:TestPoint_Pad_D1.5mm, F.Cu at (155.8, 144.6)
- added TP7: SCL TP, TestPoint:TestPoint_Keystone_5000-5004_Miniature, F.Cu at (148.7, 112.0)
- added TP8: SDA TP, TestPoint:TestPoint_Keystone_5000-5004_Miniature, F.Cu at (141.9, 101.9)
- added TP9: GPS-TX-UART TP, TestPoint:TestPoint_Keystone_5000-5004_Miniature, F.Cu at (143.3, 98.7)
- added U5: XTSD04GLGEAG, Exo_Bronco_Avionics_Footprints:SON127P600X800X95-8N, B.Cu at (171.2, 109.8)
- added kibuzzard-6562B80B: G***, kibuzzard-6562B80B, F.Cu at (144.6, 82.0)
- added kibuzzard-6562B89C: G***, kibuzzard-6562B89C, F.Cu at (143.7, 86.7)
- added kibuzzard-6562B902: G***, kibuzzard-6562B902, F.Cu at (148.8, 114.8)
- added kibuzzard-6562B960: G***, kibuzzard-6562B960, F.Cu at (138.0, 102.0)
- added kibuzzard-6562B97E: G***, kibuzzard-6562B97E, F.Cu at (147.3, 86.7)
- added kibuzzard-6562B984: G***, kibuzzard-6562B984, F.Cu at (139.8, 98.7)
- added kibuzzard-6562F408: G***, kibuzzard-6562F408, F.Cu at (124.3, 70.8)
- added kibuzzard-6562F5B5: G***, kibuzzard-6562F5B5, F.Cu at (160.0, 147.6)
- TP1: value TestPoint -> Vbatt TP
- moved kibuzzard-640E8E65 40.9 mm to (169.2, 151.0)
- moved G*** 13.9 mm to (140.6, 154.0)
- moved C4 11.7 mm to (151.7, 120.6), turned to 180 degrees
- moved kibuzzard-6400F0D2 7.53 mm to (173.3, 69.0)
- moved kibuzzard-63F7FEBE 6.45 mm to (126.1, 114.3), turned to 0 degrees
- moved kibuzzard-63F7FA90 5.61 mm to (172.9, 100.6)
- moved G*** 3.16 mm to (141.5, 136.0)
- moved SW1 0.27 mm to (171.3, 107.7)
- moved TP1 0.18 mm to (164.2, 128.2)
- moved BZ1 0.07 mm to (156.0, 114.7), turned to 90 degrees
Connections:
- net Net-(R10-Pad2) renamed Vbatt TP
- IC1 pad 15: unconnected-(IC1-IO3-Pad15) -> AIO3/XTSD_CS
- IC1 pad 26: unconnected-(IC1-IO45-Pad26) -> IO45/TDO
- R6 pad 1: IO40/TDO -> IO45/TDO
- U4 pad 2: IO40/TDO -> IO45/TDO
Routing:
- net IO45/TDO: track 0.00 -> 67.3 mm, vias 0 -> 2
- net SPICLK: track 82.3 -> 125.7 mm, vias 3 -> 6
- net AIO3/XTSD_CS: track 0.00 -> 37.8 mm, vias 0 -> 1
- net SPIQ: track 84.0 -> 116.3 mm, vias 3 -> 6
- net SPID: track 89.7 -> 117.9 mm, vias 3 -> 6
- net +3V3: track 65.6 -> 76.3 mm, vias 24 -> 25
- net A3: track 64.1 -> 69.0 mm
- net A2: track 67.9 -> 72.7 mm
- net A4: track 60.3 -> 65.1 mm
- net TX: track 35.3 -> 39.8 mm
- net +5V: track 91.7 -> 96.2 mm
- net VBUS: track 24.3 -> 28.5 mm
- net MFET3: track 96.0 -> 99.7 mm
- net MFET2: track 88.6 -> 92.2 mm
- net MFET1: track 81.0 -> 84.6 mm
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Other:
- outline, holes or cut-outs redrawn
- board text added: "3V3"
- board text added: "A1"
- board text added: "Aivie Quinto | Marilyn Hernandez Aaron De Castro | John Tran | Liz Woo Raphael Napinas | Tom Solomon"
- board text added: "Dad 1: Tim Bogman & Dad 2: Antony Makar"
- board text added: "MFET1 A4"
- board text added: "MFET2 A3"
- board text added: "MFET3 A2"
- board text added: "MFET4"
- board text added: "PYRO_HPO"
- board text added: "RG5v"
- board text added: "VBATT"
- board text added: "VBUS"
- board text removed: "Tim Bogman | Antony Makar | Zee Mahafey Kevin Foyet | Daniel Pasion | Luc Saikali Priytham Sai Chand"
