File: Sprinkle/AvionicsV0.kicad_sch (KiCad schematic)
At the start: 0 parts

Commit message: Add files via upload
Other:
- sheet Storage renamed Storage & Test Points
Changed lines of the file:
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@@
 (kicad_sch (version 20230121) (generator eeschema)
   (paper "A4")
-  (sheet (at 128.27 113.665) (size 38.735 26.035)
+  (sheet (at 127 98.425) (size 38.735 26.035)
     (stroke (width 0.1524) (type solid))
     (fill (color 0 0 0 0.0000))
-    (property "Sheetname" "PYRO" (at 137.16 114.3 0)
+    (property "Sheetname" "PYRO" (at 135.89 99.06 0)
       (effects (font (size 5 5)) (justify left bottom))
     )
-    (property "Sheetfile" "PYRO.kicad_sch" (at 128.27 140.2846 0)
+    (property "Sheetfile" "PYRO.kicad_sch" (at 127 125.0446 0)
       (effects (font (size 1.27 1.27)) (justify left top))
     )
@@
     )
   )
-  (sheet (at 52.7558 113.5126) (size 38.1 25.4)
+  (sheet (at 51.4858 98.2726) (size 38.1 25.4)
     (stroke (width 0.1524) (type solid))
     (fill (color 0 0 0 0.0000))
-    (property "Sheetname" "Connectors" (at 51.181 114.681 0)
+    (property "Sheetname" "Connectors" (at 49.911 99.441 0)
       (effects (font (size 5 5)) (justify left bottom))
     )
-    (property "Sheetfile" "Connectors.kicad_sch" (at 52.7558 139.4972 0)
+    (property "Sheetfile" "Connectors.kicad_sch" (at 51.4858 124.2572 0)
       (effects (font (size 1.27 1.27)) (justify left top))
     )
@@
     )
   )
-  (sheet (at 205.0796 109.855) (size 38.1 25.4)
+  (sheet (at 203.8096 98.425) (size 38.1 25.4)
     (stroke (width 0.1524) (type solid))
     (fill (color 0 0 0 0.0000))
-    (property "Sheetname" "Sensors" (at 209.5246 111.125 0)
+    (property "Sheetname" "Sensors" (at 208.2546 99.695 0)
       (effects (font (size 5 5)) (justify left bottom))
     )
-    (property "Sheetfile" "Sensors.kicad_sch" (at 205.3082 135.8646 0)
+    (property "Sheetfile" "Sensors.kicad_sch" (at 204.0382 124.4346 0)
       (effects (font (size 1.27 1.27)) (justify left top))
     )
@@
     )
   )
-  (sheet (at 53.34 162.56) (size 36.83 26.67) (fields_autoplaced)
+  (sheet (at 50.8 149.86) (size 36.83 26.67)
     (stroke (width 0.1524) (type solid))
     (fill (color 0 0 0 0.0000))
-    (property "Sheetname" "Storage" (at 53.34 161.8484 0)
-      (effects (font (size 1.27 1.27)) (justify left bottom))
+    (property "Sheetname" "Storage & Test Points" (at 34.29 148.59 0)
+      (effects (font (size 4.27 4.27)) (justify left bottom))
     )
-    (property "Sheetfile" "untitled.kicad_sch" (at 53.34 189.8146 0)
+    (property "Sheetfile" "untitled.kicad_sch" (at 50.8 177.1146 0)
       (effects (font (size 1.27 1.27)) (justify left top))
     )
