File: Sprinkle/GPS.kicad_sch (KiCad schematic)
At the start: 12 parts, among them J13 Conn_Coaxial, U4 FGPMMOPA6H

Commit message: Add files via upload
Connections:
- net IO40/TDO renamed IO45/TDO
Changed lines of the file:
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@@
     )
   )
-  (global_label "IO40{slash}TDO" (shape input) (at 154.94 83.82 180) (fields_autoplaced)
+  (global_label "IO45{slash}TDO" (shape input) (at 154.94 83.82 180) (fields_autoplaced)
     (effects (font (size 1.27 1.27)) (justify right))
-    (property "Intersheetrefs" "${INTERSHEET_REFS}" (at 143.3629 83.7406 0)
+    (property "Intersheetrefs" "${INTERSHEET_REFS}" (at 143.3561 83.82 0)
       (effects (font (size 1.27 1.27)) (justify right) hide)
     )
