File: Sprinkle/Power.kicad_sch (KiCad schematic)
At the start: 26 parts, among them IC3 NCP1117IST33T3G, J3 Conn_01x02, M1 TP6841S6-A

Commit message: Add files via upload
Parts:
- removed TP1: TestPoint, TestPoint:TestPoint_Pad_D1.5mm, symbol Connector:TestPoint
Connections:
- net Vbatt TP: now reaches R10.2, R11.1, R13.2
Changed lines of the file:
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@@
-    (stroke (width 0) (type default))
-  )
-  (wire (pts (xy 144.78 168.91) (xy 154.94 168.91))
     (stroke (width 0) (type default))
   )
@@
   )
   (wire (pts (xy 218.44 76.2) (xy 231.775 76.2))
+    (stroke (width 0) (type default))
+  )
+  (wire (pts (xy 144.78 168.91) (xy 149.86 168.91))
     (stroke (width 0) (type default))
   )
@@
   (text "Power" (at 13.8176 21.0312 0)
     (effects (font (size 5 5)) (justify left bottom))
+  )
+  (global_label "Vbatt TP" (shape input) (at 149.86 168.91 0) (fields_autoplaced)
+    (effects (font (size 1.27 1.27)) (justify left))
+    (property "Intersheetrefs" "${INTERSHEET_REFS}" (at 160.1548 168.91 0)
+      (effects (font (size 1.27 1.27)) (justify left) hide)
+    )
   )
   (global_label "RG5v" (shape input) (at 41.91 151.13 180) (fields_autoplaced)
@@
         )
       )
-    )
-  )
-  (symbol (lib_id "Connector:TestPoint") (at 154.94 168.91 270) (unit 1)
-    (in_bom yes) (on_board yes) (dnp no) (fields_autoplaced)
-    (property "Reference" "TP1" (at 160.02 167.6399 90)
-      (effects (font (size 1.27 1.27)) (justify left))
-    )
-    (property "Value" "TestPoint" (at 160.02 170.1799 90)
-      (effects (font (size 1.27 1.27)) (justify left))
-    )
-    (property "Footprint" "TestPoint:TestPoint_Pad_D1.5mm" (at 154.94 173.99 0)
-      (effects (font (size 1.27 1.27)) hide)
-    )
-    (property "Datasheet" "~" (at 154.94 173.99 0)
-      (effects (font (size 1.27 1.27)) hide)
-    )
-    (pin "1")
-    (instances
-      (project "AvionicsV0"
-        (path "/e63e39d7-6ac0-4ffd-8aa3-1841a4541b55/67bc02c4-8903-4c53-b030-82afb6b77135"
-          (reference "TP1") (unit 1)
-        )
-      )
