File: Sprinkle/untitled.kicad_sch (KiCad schematic)
At the start: 2 parts, among them U5 XTSD04GLGEAG

Commit message: Add files via upload
Parts:
- removed U5: XTSD04GLGEAG, SON127P600X800X95-8N, symbol XTSD04GLGEAG:XTSD04GLGEAG
- added R8: 10k, Resistor_SMD:R_0603_1608Metric, symbol Device:R
- added TP1: Vbatt TP, TestPoint:TestPoint_Pad_D1.5mm, symbol Connector:TestPoint
- added TP10: GPS-RX-UART-TP, TestPoint:TestPoint_Keystone_5000-5004_Miniature, symbol Connector:TestPoint
- added TP13: SPI-MISO, TestPoint:TestPoint_Keystone_5000-5004_Miniature, symbol Connector:TestPoint
- added TP14: SPI-MOSI, TestPoint:TestPoint_Keystone_5000-5004_Miniature, symbol Connector:TestPoint
- added TP15: SPI-CLK, TestPoint:TestPoint_Keystone_5000-5004_Miniature, symbol Connector:TestPoint
- added TP16: Pyro-MFET4-TP, TestPoint:TestPoint_Pad_D1.0mm, symbol Connector:TestPoint
- added TP17: Pyro-MFET1-TP, TestPoint:TestPoint_Pad_D1.0mm, symbol Connector:TestPoint
- added TP18, TP19: Pyro-MFET2-TP, TestPoint:TestPoint_Pad_D1.0mm, symbol Connector:TestPoint
- added TP2: GND TP, TestPoint:TestPoint_Keystone_5000-5004_Miniature, symbol Connector:TestPoint
- added TP20: Pyro-HPO-TP, TestPoint:TestPoint_Pad_D1.0mm, symbol Connector:TestPoint
- added TP21: Cont-A4-TP, TestPoint:TestPoint_Pad_D1.0mm, symbol Connector:TestPoint
- added TP22: Cont-A3-TP, TestPoint:TestPoint_Pad_D1.0mm, symbol Connector:TestPoint
- added TP23: Cont-A2-TP, TestPoint:TestPoint_Pad_D1.0mm, symbol Connector:TestPoint
- added TP24: Cont-A1-TP, TestPoint:TestPoint_Pad_D1.0mm, symbol Connector:TestPoint
- added TP3: 3V3 TP, TestPoint:TestPoint_Pad_D1.5mm, symbol Connector:TestPoint
- added TP4: 5V TP, TestPoint:TestPoint_Pad_D1.5mm, symbol Connector:TestPoint
- added TP5: Vbus TP, TestPoint:TestPoint_Pad_D1.5mm, symbol Connector:TestPoint
- added TP6: RG5 TP, TestPoint:TestPoint_Pad_D1.5mm, symbol Connector:TestPoint
- added TP7: SCL TP, TestPoint:TestPoint_Keystone_5000-5004_Miniature, symbol Connector:TestPoint
- added TP8: SDA TP, TestPoint:TestPoint_Keystone_5000-5004_Miniature, symbol Connector:TestPoint
- added TP9: GPS-TX-UART TP, TestPoint:TestPoint_Keystone_5000-5004_Miniature, symbol Connector:TestPoint
- added U5: XTSD04GLGEAG, Exo_Bronco_Avionics_Footprints:SON127P600X800X95-8N, symbol EXO_BRONCO_Avionics_Sym:XTSD04GLGEAG
- C17: footprint (none) -> Capacitor_SMD:C_0603_1608Metric
Connections:
- net +3V3: now also R8.1, TP3.1, U5.8 (VDD)
- net GND: now also TP2.1, U5.4 (VSS)
- net SPICLK: now also TP15.1, U5.3 (CLK)
- net SPID: now also TP14.1, U5.5 (CMD/DI)
- net SPIQ: now also TP13.1, U5.6 (SD0/DO)
- new net +5V: TP4.1
- new net A1: TP24.1
- new net A2: TP23.1
- new net A3: TP22.1
- new net A4: TP21.1
- new net AIO3/XTSD_CS: R8.2, U5.2 (SD3/~{CS})
- new net MFET1: TP17.1
- new net MFET2: TP18.1
- new net MFET3: TP19.1
- new net MFET4: TP16.1
- new net PYRO_HPO: TP20.1
- new net RG5v: TP6.1
- new net RX: TP10.1
- new net SCL: TP7.1
- new net SDA: TP8.1
- new net TX: TP9.1
- new net VBUS: TP5.1
- new net Vbatt TP: TP1.1
Other:
- note added: "Power TP"
- note added: "Pyro Continuity TP"
- note added: "Pyro TP"
- note added: "Signal TP"
- note added: "Test Points"
- note removed: "FINISH WITH CS line!!!!"
- moved on the sheet: C17
